Commit message: issues resolved with link_00

File: plotter/plotter_description/urdf/plotterv2.xacro (robot description, xacro)
@@ -7,4 +7,15 @@
     <!-- END - Include -->
     <!-- BGN - Robot description -->
+    <link name="world" />
+    <joint name="world__link_00" type="fixed">
+        <parent link="world"/>
+        <child link="${link_00_name}"/>
+    </joint>
+    <link name="${link_00_name}" />
+    <joint name="${link_00_name}__${link_01_name}" type="fixed">
+        <parent link="${link_00_name}"/>
+        <child link="${link_01_name}"/>
+    </joint>
+    <!--
     <xacro:m_link_box name="${link_00_name}" origin_rpy="0 0 0" origin_xyz = "0 0 0"
               mass = "1024"
@@ -13,7 +24,16 @@
               izz = "170.67"
               size = "0.032 0.004 0.068" />
+    <xacro:m_joint name="${link_00_name}__${link_01_name}" type="fixed"
+	axis_xyz = "0 0 1"
+	origin_rpy ="0 0 0" origin_xyz = "0 ${0.004/2} 0"
+        parent = "${link_00_name}"  child = "${link_01_name}"
+        limit_e = "1000.0"
+        limit_l = "-1.57"
+        limit_u = "1.57"
+        limit_v = "0.5" />
     <xacro:m_joint_fixed name="${link_00_name}__${link_01_name}" type="fixed"
        origin_rpy ="0 0 0" origin_xyz = "0 ${0.004/2} 0"
        parent = "${link_00_name}"  child = "${link_01_name}" />
+-->
     <xacro:m_link_box name="${link_01_name}" origin_rpy="0 0 0" origin_xyz="0 ${0.036/2 } 0"
         size = "0.02 0.036 0.045"
@@ -53,5 +73,4 @@
             <plugin name="gazebo_ros_control" filename="libgazebo_ros_control.so">
                 <robotNamespace>/plotter</robotNamespace>
-		<robotSimType>gazebo_ros_control/DefaultRobotHWSim</robotSimType>
             </plugin>
         </gazebo>

File: plotter/plotter_description/urdf/plotterv2_gen.urdf (robot description, URDF)
Before this commit: robot plotter, 4 links, 3 joints
Joints:
- joint link_00__link_01: axis (none) -> 0 0 1; limit (none) -> lower=-1.57 upper=1.57 effort=1000.0 velocity=0.5

File: plotter/plotter_description/urdf/robot_parameters.xacro (robot description, xacro)
@@ -5,5 +5,3 @@
   <xacro:property name="link_02_name" value="link_02" />
   <xacro:property name="link_03_name" value="link_03" />
-  <xacro:property name="link_04_name" value="link_04" />
-  <xacro:property name="link_05_name" value="link_05" />
 </robot>

Commit message: improvements

File: plotter/plotter_description/urdf/plotterv2.xacro (robot description, xacro)
@@ -8,8 +8,9 @@
     <!-- BGN - Robot description -->
     <link name="world" />
-    <joint name="world__link_00" type="fixed">
+    <joint name="world__link_01" type="fixed">
         <parent link="world"/>
-        <child link="${link_00_name}"/>
+        <child link="${link_01_name}"/>
     </joint>
+    <!--
     <link name="${link_00_name}" />
     <joint name="${link_00_name}__${link_01_name}" type="fixed">
@@ -17,5 +18,4 @@
         <child link="${link_01_name}"/>
     </joint>
-    <!--
     <xacro:m_link_box name="${link_00_name}" origin_rpy="0 0 0" origin_xyz = "0 0 0"
               mass = "1024"
