Commit message: actualizacion 1tb

File: plotter/plotter_description/urdf/links_joints.xacro (robot description, xacro)
@@ -12,8 +12,8 @@
       <type>transmission_interface/SimpleTransmission</type>
       <joint name="${name}">
-        <hardwareInterface>hardware_interface/EffortJointInterface</hardwareInterface>
+        <hardwareInterface>hardware_interface/PositionJointInterface</hardwareInterface>
       </joint>
       <actuator name="motor_${name}">
-        <hardwareInterface>hardware_interface/EffortJointInterface</hardwareInterface>
+        <hardwareInterface>hardware_interface/PositionJointInterface</hardwareInterface>
         <mechanicalReduction>1</mechanicalReduction>
       </actuator>
@@ -29,8 +29,8 @@
       <type>transmission_interface/SimpleTransmission</type>
       <joint name="${name}">
-        <hardwareInterface>hardware_interface/EffortJointInterface</hardwareInterface>
+        <hardwareInterface>hardware_interface/PositionJointInterface</hardwareInterface>
       </joint>
       <actuator name="motor_${name}">
-        <hardwareInterface>hardware_interface/EffortJointInterface</hardwareInterface>
+        <hardwareInterface>hardware_interface/PositionJointInterface</hardwareInterface>
         <mechanicalReduction>1</mechanicalReduction>
       </actuator>

File: plotter/plotter_description/urdf/plotterv2.xacro (robot description, xacro)
@@ -36,41 +36,45 @@
        parent = "${link_00_name}"  child = "${link_01_name}" />
 -->
-    <xacro:m_link_box name="${link_01_name}" origin_rpy="0 0 0" origin_xyz="0 ${0.036/2 } 0"
+    <xacro:m_link_box name="${link_01_name}" origin_rpy="0 0 0"
+        origin_xyz="0 ${0.036/2 } 0.2"
         size = "0.02 0.036 0.045"
-        mass = "1024"
-        ixx = "170.667" ixy = "0" ixz = "0"
-        iyy = "170.67"  iyz = "0"
-        izz = "170.67" />
+        mass = "0.01"
+        ixx = "0.4" ixy = "0" ixz = "0"
+        iyy = "0.4"  iyz = "0"
+        izz = "0.4" />
     <xacro:m_joint name="${link_01_name}__${link_02_name}" type="revolute"
         axis_xyz = "0 0 1"
-        origin_rpy ="0 0 0" origin_xyz = "0 0.036 0"
+        origin_rpy ="0 0 0" origin_xyz = "0 0.036 0.2"
         parent = "${link_01_name}"  child = "${link_02_name}"
-        limit_e = "1000.0"
+        limit_e = "3.0"
         limit_l = "-1.57"
         limit_u = "1.57"
         limit_v = "0.5" />
-    <xacro:m_link_box name="${link_02_name}" origin_rpy="0 0 0" origin_xyz="0 ${0.061/2} 0"
+    <xacro:m_link_box name="${link_02_name}" origin_rpy="0 0 0"
+        origin_xyz="0 ${0.061/2} 0"
         size = "0.02 0.061 0.057"
-        mass = "1024"
-        ixx = "170.667" ixy = "0" ixz = "0"
-        iyy = "170.67"  iyz = "0"
-        izz = "170.67" />
+        mass = "0.01"
+        ixx = "0.4" ixy = "0" ixz = "0"
+        iyy = "0.4"  iyz = "0"
+        izz = "0.4" />
     <xacro:m_joint name="${link_02_name}__${link_03_name}" type="revolute"
         axis_xyz = "0 0 1"
         origin_rpy ="0 0 0" origin_xyz = "0 0.061 0"
         parent = "${link_02_name}"  child = "${link_03_name}"
-        limit_e = "1000.0"
+        limit_e = "3.0"
         limit_l = "-1.57"
         limit_u = "1.57"
         limit_v = "0.5" />
-    <xacro:m_link_box name="${link_03_name}" origin_rpy="0 0 0" origin_xyz="0 ${0.026/2} 0"
+    <xacro:m_link_box name="${link_03_name}" origin_rpy="0 0 0"
+        origin_xyz="0 ${0.026/2} 0"
         size = "0.02 0.026 0.057"
-        mass = "1024"
-        ixx = "170.667" ixy = "0" ixz = "0"
-        iyy = "170.67"  iyz = "0"
-        izz = "170.67" />
+        mass = "0.01"
+        ixx = "0.4" ixy = "0" ixz = "0"
+        iyy = "0.4"  iyz = "0"
+        izz = "0.4" />
         <gazebo>
             <plugin name="gazebo_ros_control" filename="libgazebo_ros_control.so">
                 <robotNamespace>/plotter</robotNamespace>
+		<robotSimType>gazebo_ros_control/DefaultRobotHWSim</robotSimType>
             </plugin>
         </gazebo>

File: plotter/plotter_description/urdf/plotterv2_gen.urdf (robot description, URDF)
Before this commit: robot plotter, 4 links, 3 joints
Links:
- removed link link_00
- added link world
- link link_01: mass 1024 -> 0.01
- link link_02: mass 1024 -> 0.01
- link link_03: mass 1024 -> 0.01
Joints:
- removed joint link_00__link_01
- added joint world__link_01: type fixed, parent world, child link_01
- joint link_01__link_02: limit lower=-1.57 upper=1.57 effort=1000.0 velocity=0.5 -> lower=-1.57 upper=1.57 effort=3.0 velocity=0.5; origin xyz=0 0.036 0 rpy=0 0 0 -> xyz=0 0.036 0.2 rpy=0 0 0
- joint link_02__link_03: limit lower=-1.57 upper=1.57 effort=1000.0 velocity=0.5 -> lower=-1.57 upper=1.57 effort=3.0 velocity=0.5
